File: MicroBitFeather.sch (KiCad schematic (older format))
At the start: 16 parts, among them J1 Feather_Long, J2 Barrel_Jack_MountingPin, J3 Feather_Short, J4 NeoPixels, J5 microbit_edge_connector, U1 74AHCT125, U2 MCP1702-3302E_TO92

Commit message: Start associating a few footprints.
Parts:
- C1: footprint (none) -> Capacitors_THT:CP_Radial_D10.0mm_P5.00mm
- C5: footprint (none) -> Capacitors_THT:CP_Radial_D6.3mm_P2.50mm
- D1: footprint (none) -> Diodes_THT:D_DO-15_P10.16mm_Horizontal
- J1: footprint (none) -> Socket_Strips:Socket_Strip_Straight_1x16_Pitch2.54mm
- J3: footprint (none) -> Socket_Strips:Socket_Strip_Straight_1x12_Pitch2.54mm
- U1: footprint (none) -> Housings_DIP:DIP-14_W7.62mm
Changed lines of the file:
@@
 F 0 "J1" H 4300 2350 60  0000 L CNN
 F 1 "Feather_Long" H 4300 2250 60  0000 L CNN
-F 2 "" H 4200 2100 60  0001 C CNN
+F 2 "Socket_Strips:Socket_Strip_Straight_1x16_Pitch2.54mm" H 4200 2100 60  0001 C CNN
 F 3 "" H 4200 2100 60  0001 C CNN
 F 4 "PPPC161LFBN-RC" H 4200 2100 60  0001 C CNN "MPN"
@@
 F 0 "J3" H 5700 2750 60  0000 L CNN
 F 1 "Feather_Short" H 5700 2650 60  0000 L CNN
-F 2 "" H 5600 2500 60  0001 C CNN
+F 2 "Socket_Strips:Socket_Strip_Straight_1x12_Pitch2.54mm" H 5600 2500 60  0001 C CNN
 F 3 "" H 5600 2500 60  0001 C CNN
 F 4 "PPPC121LFBN-RC" H 5600 2500 60  0001 C CNN "MPN"
@@
 Connection ~ 7150 4200
 $Comp
-L +3V3 #PWR14
+L +3V3 #PWR01
 U 1 1 5B877C6E
 P 7000 4000
-F 0 "#PWR14" H 7000 3850 50  0001 C CNN
+F 0 "#PWR01" H 7000 3850 50  0001 C CNN
 F 1 "+3V3" H 7000 4140 50  0000 C CNN
 F 2 "" H 7000 4000 50  0001 C CNN
@@
 Connection ~ 7150 5000
 $Comp
-L GND #PWR15
+L GND #PWR02
 U 1 1 5B877F3E
 P 7000 4900
-F 0 "#PWR15" H 7000 4650 50  0001 C CNN
+F 0 "#PWR02" H 7000 4650 50  0001 C CNN
 F 1 "GND" H 7000 4750 50  0000 C CNN
 F 2 "" H 7000 4900 50  0001 C CNN
@@
 $EndComp
 $Comp
-L +3V3 #PWR3
+L +3V3 #PWR03
 U 1 1 5B87818E
 P 3600 1900
-F 0 "#PWR3" H 3600 1750 50  0001 C CNN
+F 0 "#PWR03" H 3600 1750 50  0001 C CNN
 F 1 "+3V3" H 3600 2040 50  0000 C CNN
 F 2 "" H 3600 1900 50  0001 C CNN
@@
 NoConn ~ 4200 2300
 $Comp
-L GND #PWR4
+L GND #PWR04
 U 1 1 5B878369
 P 3600 2500
-F 0 "#PWR4" H 3600 2250 50  0001 C CNN
+F 0 "#PWR04" H 3600 2250 50  0001 C CNN
 F 1 "GND" H 3600 2350 50  0000 C CNN
 F 2 "" H 3600 2500 50  0001 C CNN
@@
 	4000 3600 4200 3600
 $Comp
-L +3V3 #PWR13
+L +3V3 #PWR05
 U 1 1 5B878A64
 P 6100 2400
-F 0 "#PWR13" H 6100 2250 50  0001 C CNN
+F 0 "#PWR05" H 6100 2250 50  0001 C CNN
 F 1 "+3V3" H 6100 2540 50  0000 C CNN
 F 2 "" H 6100 2400 50  0001 C CNN
@@
 	5600 2600 5800 2600
 $Comp
-L +5V #PWR10
+L +5V #PWR06
 U 1 1 5B878BFE
 P 5700 2400
-F 0 "#PWR10" H 5700 2250 50  0001 C CNN
+F 0 "#PWR06" H 5700 2250 50  0001 C CNN
 F 1 "+5V" H 5700 2540 50  0000 C CNN
 F 2 "" H 5700 2400 50  0001 C CNN
@@
 FIXME: Check pinout!
 $Comp
-L GND #PWR12
+L GND #PWR07
 U 1 1 5B87949E
 P 5850 5000
-F 0 "#PWR12" H 5850 4750 50  0001 C CNN
+F 0 "#PWR07" H 5850 4750 50  0001 C CNN
 F 1 "GND" H 5850 4850 50  0000 C CNN
 F 2 "" H 5850 5000 50  0001 C CNN
@@
 $EndComp
 $Comp
-L +5V #PWR11
+L +5V #PWR08
 U 1 1 5B8794C4
 P 5850 4550
-F 0 "#PWR11" H 5850 4400 50  0001 C CNN
+F 0 "#PWR08" H 5850 4400 50  0001 C CNN
 F 1 "+5V" H 5850 4690 50  0000 C CNN
 F 2 "" H 5850 4550 50  0001 C CNN
@@
 F 0 "U1" H 4450 5450 50  0000 C CNN
 F 1 "74AHCT125" H 4950 4150 50  0000 C CNN
-F 2 "" H 4700 4800 60  0000 C CNN
+F 2 "Housings_DIP:DIP-14_W7.62mm" H 4700 4800 60  0001 C CNN
 F 3 "" H 4700 4800 60  0000 C CNN
 F 4 "SN74AHCT125N" H 4700 4800 60  0001 C CNN "MPN"
@@
 $EndComp
 $Comp
-L +5V #PWR6
+L +5V #PWR09
 U 1 1 5B87920C
 P 4700 4000
-F 0 "#PWR6" H 4700 3850 50  0001 C CNN
+F 0 "#PWR09" H 4700 3850 50  0001 C CNN
 F 1 "+5V" H 4700 4140 50  0000 C CNN
 F 2 "" H 4700 4000 50  0001 C CNN
@@
 $EndComp
 $Comp
-L GND #PWR7
+L GND #PWR010
 U 1 1 5B879238
 P 4700 5600
-F 0 "#PWR7" H 4700 5350 50  0001 C CNN
+F 0 "#PWR010" H 4700 5350 50  0001 C CNN
 F 1 "GND" H 4700 5450 50  0000 C CNN
 F 2 "" H 4700 5600 50  0001 C CNN
@@
 	4700 5500 4700 5600
 $Comp
-L +5V #PWR8
+L +5V #PWR011
 U 1 1 5B879F10
 P 4900 6000
-F 0 "#PWR8" H 4900 5850 50  0001 C CNN
+F 0 "#PWR011" H 4900 5850 50  0001 C CNN
 F 1 "+5V" H 4900 6140 50  0000 C CNN
 F 2 "" H 4900 6000 50  0001 C CNN
@@
 $EndComp
 $Comp
-L GND #PWR5
+L GND #PWR012
 U 1 1 5B879F3C
 P 4500 6700
-F 0 "#PWR5" H 4500 6450 50  0001 C CNN
+F 0 "#PWR012" H 4500 6450 50  0001 C CNN
 F 1 "GND" H 4500 6550 50  0000 C CNN
 F 2 "" H 4500 6700 50  0001 C CNN
@@
 Connection ~ 6200 6600
 $Comp
-L +3V3 #PWR16
+L +3V3 #PWR013
 U 1 1 5B87BEFA
 P 7600 6000
-F 0 "#PWR16" H 7600 5850 50  0001 C CNN
+F 0 "#PWR013" H 7600 5850 50  0001 C CNN
 F 1 "+3V3" H 7600 6140 50  0000 C CNN
 F 2 "" H 7600 6000 50  0001 C CNN
@@
 F 0 "D1" H 7200 6200 50  0000 C CNN
 F 1 "D_Schottky" H 7200 6000 50  0000 C CNN
-F 2 "" H 7200 6100 50  0001 C CNN
+F 2 "Diodes_THT:D_DO-15_P10.16mm_Horizontal" H 7200 6100 50  0001 C CNN
 F 3 "" H 7200 6100 50  0001 C CNN
 F 4 "SB240TA" H 7200 6100 60  0001 C CNN "MPN"
@@
 F 0 "C5" H 7625 6450 50  0000 L CNN
 F 1 "47µF" H 7625 6250 50  0000 L CNN
-F 2 "" H 7638 6200 50  0001 C CNN
+F 2 "Capacitors_THT:CP_Radial_D6.3mm_P2.50mm" H 7638 6200 50  0001 C CNN
 F 3 "" H 7600 6350 50  0001 C CNN
 F 4 "ECE-A1CKS470" H 7600 6350 60  0001 C CNN "MPN"
@@
 $EndComp
 $Comp
-L GND #PWR9
+L GND #PWR014
 U 1 1 5B87CC46
 P 5350 4100
-F 0 "#PWR9" H 5350 3850 50  0001 C CNN
+F 0 "#PWR014" H 5350 3850 50  0001 C CNN
 F 1 "GND" H 5350 3950 50  0000 C CNN
 F 2 "" H 5350 4100 50  0001 C CNN
@@
 F 0 "C1" H 3325 4750 50  0000 L CNN
 F 1 "1000µF" H 3325 4550 50  0000 L CNN
-F 2 "" H 3300 4650 50  0001 C CNN
+F 2 "Capacitors_THT:CP_Radial_D10.0mm_P5.00mm" H 3300 4650 50  0001 C CNN
 F 3 "" H 3300 4650 50  0001 C CNN
 F 4 "10WXA1000MEFCT810X9" H 3300 4650 60  0001 C CNN "MPN"
@@
 $EndComp
 $Comp
-L GND #PWR2
+L GND #PWR015
 U 1 1 5B87D3B2
 P 3300 4900
-F 0 "#PWR2" H 3300 4650 50  0001 C CNN
+F 0 "#PWR015" H 3300 4650 50  0001 C CNN
 F 1 "GND" H 3300 4750 50  0000 C CNN
 F 2 "" H 3300 4900 50  0001 C CNN
@@
 $EndComp
 $Comp
-L +5V #PWR1
+L +5V #PWR016
 U 1 1 5B87D3F6
 P 3300 4400
-F 0 "#PWR1" H 3300 4250 50  0001 C CNN
+F 0 "#PWR016" H 3300 4250 50  0001 C CNN
 F 1 "+5V" H 3300 4540 50  0000 C CNN
 F 2 "" H 3300 4400 50  0001 C CNN
@@
 	3300 4800 3300 4900
 $Comp
-L PWR_FLAG #FLG1
+L PWR_FLAG #FLG017
 U 1 1 5B87DB70
 P 5200 6000
-F 0 "#FLG1" H 5200 6075 50  0001 C CNN
+F 0 "#FLG017" H 5200 6075 50  0001 C CNN
 F 1 "PWR_FLAG" H 5200 6150 50  0000 C CNN
 F 2 "" H 5200 6000 50  0001 C CNN
@@
 $EndComp
 $Comp
-L PWR_FLAG #FLG2
+L PWR_FLAG #FLG018
 U 1 1 5B87DBB4
 P 8000 6000
-F 0 "#FLG2" H 8000 6075 50  0001 C CNN
+F 0 "#FLG018" H 8000 6075 50  0001 C CNN
 F 1 "PWR_FLAG" H 8000 6150 50  0000 C CNN
 F 2 "" H 8000 6000 50  0001 C CNN
@@
 $EndComp
 $Comp
-L PWR_FLAG #FLG3
+L PWR_FLAG #FLG019
 U 1 1 5B87DBF8
 P 8000 6500
-F 0 "#FLG3" H 8000 6575 50  0001 C CNN
+F 0 "#FLG019" H 8000 6575 50  0001 C CNN
 F 1 "PWR_FLAG" H 8000 6650 50  0000 C CNN
 F 2 "" H 8000 6500 50  0001 C CNN

Commit message: Finish footprint associations.
Parts:
- C2, C3, C4: footprint (none) -> Capacitors_THT:C_Rect_L7.0mm_W2.5mm_P5.00mm
- J2: footprint (none) -> footprints:BarrelJack_CUI_PJ-063AH_Horizontal_CircularHoles
- J4: footprint (none) -> Connectors_JST:JST_PH_S3B-PH-K_03x2.00mm_Angled
- J5: footprint (none) -> footprints:4UCON_10156_90deg
- R1, R2, R3: footprint (none) -> Resistors_THT:R_Axial_DIN0207_L6.3mm_D2.5mm_P7.62mm_Horizontal
Changed lines of the file:
@@
 F 0 "J5" H 7750 5350 50  0000 C CNN
 F 1 "microbit_edge_connector" H 7750 5250 50  0000 C CNN
-F 2 "" H 7600 3200 50  0001 C CNN
+F 2 "footprints:4UCON_10156_90deg" H 7600 3200 50  0001 C CNN
 F 3 "" H 7600 3200 50  0001 C CNN
 F 4 "3342" H 7700 3300 60  0001 C CNN "MPN"
@@
 F 0 "R1" V 3930 2000 50  0000 C CNN
 F 1 "10K" V 3850 2000 50  0000 C CNN
-F 2 "" V 3780 2000 50  0001 C CNN
+F 2 "Resistors_THT:R_Axial_DIN0207_L6.3mm_D2.5mm_P7.62mm_Horizontal" V 3780 2000 50  0001 C CNN
 F 3 "" H 3850 2000 50  0001 C CNN
 F 4 "CF14JT10K0" H 3850 2000 60  0001 C CNN "MPN"
@@
 F 0 "J4" H 6400 5000 50  0000 C CNN
 F 1 "NeoPixels" H 6400 4600 50  0000 C CNN
-F 2 "" H 6400 4800 50  0001 C CNN
+F 2 "Connectors_JST:JST_PH_S3B-PH-K_03x2.00mm_Angled" H 6400 4800 50  0001 C CNN
 F 3 "" H 6400 4800 50  0001 C CNN
 F 4 "S3B-PH-K-S(LF)(SN)" H 6400 4800 60  0001 C CNN "MPN"
@@
 F 0 "J2" H 4500 6410 50  0000 C CNN
 F 1 "Barrel_Jack_MountingPin" H 4550 5950 50  0000 L CNN
-F 2 "" H 4550 6160 50  0001 C CNN
+F 2 "footprints:BarrelJack_CUI_PJ-063AH_Horizontal_CircularHoles" H 4550 6160 50  0001 C CNN
 F 3 "" H 4550 6160 50  0001 C CNN
 F 4 "PJ-063AH" H 4500 6200 60  0001 C CNN "MPN"
@@
 F 0 "R2" V 5580 4550 50  0000 C CNN
 F 1 "470" V 5500 4550 50  0000 C CNN
-F 2 "" V 5430 4550 50  0001 C CNN
+F 2 "Resistors_THT:R_Axial_DIN0207_L6.3mm_D2.5mm_P7.62mm_Horizontal" V 5430 4550 50  0001 C CNN
 F 3 "" H 5500 4550 50  0001 C CNN
 F 4 "CF14JT470R" H 5500 4550 60  0001 C CNN "MPN"
@@
 F 0 "C3" H 5675 6450 50  0000 L CNN
 F 1 "1µF" H 5675 6250 50  0000 L CNN
-F 2 "" H 5688 6200 50  0001 C CNN
+F 2 "Capacitors_THT:C_Rect_L7.0mm_W2.5mm_P5.00mm" H 5688 6200 50  0001 C CNN
 F 3 "" H 5650 6350 50  0001 C CNN
 F 4 "K105Z20Y5VF5TH5" H 5650 6350 60  0001 C CNN "MPN"
@@
 F 0 "C2" H 5125 4150 50  0000 L CNN
 F 1 "0.1µF" H 5125 3950 50  0000 L CNN
-F 2 "" H 5138 3900 50  0001 C CNN
+F 2 "Capacitors_THT:C_Rect_L7.0mm_W2.5mm_P5.00mm" H 5138 3900 50  0001 C CNN
 F 3 "" H 5100 4050 50  0001 C CNN
 F 4 "K104K10X7RF5UH5" H 5100 4050 60  0001 C CNN "MPN"
@@
 F 0 "C4" H 6675 6450 50  0000 L CNN
 F 1 "1µF" H 6675 6250 50  0000 L CNN
-F 2 "" H 6688 6200 50  0001 C CNN
+F 2 "Capacitors_THT:C_Rect_L7.0mm_W2.5mm_P5.00mm" H 6688 6200 50  0001 C CNN
 F 3 "" H 6650 6350 50  0001 C CNN
 F 4 "K105Z20Y5VF5TH5" H 6650 6350 60  0001 C CNN "MPN"
@@
 F 0 "R3" V 6030 2600 50  0000 C CNN
 F 1 "10K" V 5950 2600 50  0000 C CNN
-F 2 "" V 5880 2600 50  0001 C CNN
+F 2 "Resistors_THT:R_Axial_DIN0207_L6.3mm_D2.5mm_P7.62mm_Horizontal" V 5880 2600 50  0001 C CNN
 F 3 "" H 5950 2600 50  0001 C CNN
 F 4 "CF14JT10K0" H 5950 2600 60  0001 C CNN "MPN"
