File: NeoBit.sch (KiCad schematic (older format))
At the start: 16 parts, among them J1 Feather_Long, J2 Barrel_Jack_MountingPin, J3 Feather_Short, J4 NeoPixels, J5 microbit_edge_connector, U1 74AHCT125, U2 MCP1702-3302E_TO92

Commit message: Add potentiometers to schematic.
Parts:
- removed J1: Feather_Long, Socket_Strips:Socket_Strip_Straight_1x16_Pitch2.54mm, symbol Feather_Long
- removed J3: Feather_Short, Socket_Strips:Socket_Strip_Straight_1x12_Pitch2.54mm, symbol Feather_Short
- removed R1, R3: 10K, Resistors_THT:R_Axial_DIN0207_L6.3mm_D2.5mm_P7.62mm_Horizontal, symbol R
- added RV? (x2): 10K, symbol R_POT_MountingPin
Connections:
- wire segments 129 -> 111
- no-connect marks 4 -> 3

Commit message: Put no-connects on most micro:bit pins.
Parts:
- gave numbers to parts that had none: 2
Connections:
- net MISO: no longer names the net of J5.33 (P14_MISO)
- net MOSI: no longer names the net of J5.31 (P15_MOSI)
- net P10: no longer names the net of J5.49 (P10)
- net P11: no longer names the net of J5.47 (P11_Button_B)
- net P12: no longer names the net of J5.45 (P12)
- net P16: no longer names the net of J5.29 (P16)
- net P3: no longer names the net of J5.79 (P3)
- net P4: no longer names the net of J5.69 (P4)
- net P5: no longer names the net of J5.67 (P5_Button_A)
- net P6: no longer names the net of J5.65 (P6)
- net P7: no longer names the net of J5.63 (P7)
- net P8: no longer names the net of J5.53 (P8)
- net P9: no longer names the net of J5.51 (P9)
- net SCK: no longer names the net of J5.35 (P13_SCK)
- net SCL: no longer names the net of J5.15 (P19_SCL)
- net SDA: no longer names the net of J5.13 (P20_SDA)
- no-connect marks 3 -> 19
Changed lines of the file:
@@
 encoding utf-8
 Sheet 1 1
-Title "Neopixel and FeatherWing adapter for Micro:Bit"
-Date "2017-08-31"
+Title "Neopixel and potentiometer adapter for Micro:Bit"
+Date "2017-09-01"
 Rev ""
 Comp "Patrick Pelletier"
@@
 	-1   0    0    1
 $EndComp
-Text Label 7000 1200 0    50   ~ 0
-P3
-Wire Wire Line
-	7000 1200 7200 1200
 Text Label 7000 1450 0    50   ~ 0
 P0
@@
 	7000 1450 7150 1450
 Connection ~ 7150 1450
-Text Label 7000 1700 0    50   ~ 0
-P4
-Text Label 7000 1800 0    50   ~ 0
-P5
-Text Label 7000 1900 0    50   ~ 0
-P6
-Text Label 7000 2000 0    50   ~ 0
-P7
 Text Label 7000 2250 0    50   ~ 0
 P1
 Wire Wire Line
-	7000 1700 7200 1700
-Wire Wire Line
-	7000 1800 7200 1800
-Wire Wire Line
-	7000 1900 7200 1900
-Wire Wire Line
-	7000 2000 7200 2000
-Wire Wire Line
 	7200 2100 7150 2100
 Wire Wire Line
@@
 	7000 2250 7150 2250
 Connection ~ 7150 2250
-Text Label 7000 2500 0    50   ~ 0
-P8
-Text Label 7000 2600 0    50   ~ 0
-P9
-Text Label 7000 2700 0    50   ~ 0
-P10
-Text Label 7000 2800 0    50   ~ 0
-P11
-Text Label 7000 2900 0    50   ~ 0
-P12
 Text Label 7000 3150 0    50   ~ 0
 P2
 Wire Wire Line
-	7000 2500 7200 2500
-Wire Wire Line
-	7000 2600 7200 2600
-Wire Wire Line
-	7000 2700 7200 2700
-Wire Wire Line
-	7000 2800 7200 2800
-Wire Wire Line
-	7000 2900 7200 2900
-Wire Wire Line
 	7200 3000 7150 3000
 Wire Wire Line
@@
 	7000 3150 7150 3150
 Connection ~ 7150 3150
-Text Label 7000 3400 0    50   ~ 0
-SCK
-Text Label 7000 3500 0    50   ~ 0
-MISO
-Text Label 7000 3600 0    50   ~ 0
-MOSI
-Text Label 7000 3700 0    50   ~ 0
-P16
-Wire Wire Line
-	7000 3400 7200 3400
-Wire Wire Line
-	7000 3500 7200 3500
-Wire Wire Line
-	7000 3600 7200 3600
-Wire Wire Line
-	7000 3700 7200 3700
 Wire Wire Line
 	7200 3800 7150 3800
@@
 	7000 4050 7150 4050
 Connection ~ 7150 4050
-Text Label 7000 4400 0    50   ~ 0
-SCL
-Text Label 7000 4500 0    50   ~ 0
-SDA
-Wire Wire Line
-	7000 4400 7200 4400
-Wire Wire Line
-	7000 4500 7200 4500
 Wire Wire Line
 	7200 4600 7150 4600
@@
 $EndComp
 $Comp
-L GND #PWR07
+L GND #PWR03
 U 1 1 5B87949E
 P 5850 5000
-F 0 "#PWR07" H 5850 4750 50  0001 C CNN
+F 0 "#PWR03" H 5850 4750 50  0001 C CNN
 F 1 "GND" H 5850 4850 50  0000 C CNN
 F 2 "" H 5850 5000 50  0001 C CNN
@@
 $EndComp
 $Comp
-L +5V #PWR08
+L +5V #PWR04
 U 1 1 5B8794C4
 P 6100 4650
-F 0 "#PWR08" H 6100 4500 50  0001 C CNN
+F 0 "#PWR04" H 6100 4500 50  0001 C CNN
 F 1 "+5V" H 6100 4790 50  0000 C CNN
 F 2 "" H 6100 4650 50  0001 C CNN
@@
 $EndComp
 $Comp
-L +5V #PWR09
+L +5V #PWR05
 U 1 1 5B87920C
 P 4700 4000
-F 0 "#PWR09" H 4700 3850 50  0001 C CNN
+F 0 "#PWR05" H 4700 3850 50  0001 C CNN
 F 1 "+5V" H 4700 4140 50  0000 C CNN
 F 2 "" H 4700 4000 50  0001 C CNN
@@
 $EndComp
 $Comp
-L GND #PWR010
+L GND #PWR06
 U 1 1 5B879238
 P 4700 5600
-F 0 "#PWR010" H 4700 5350 50  0001 C CNN
+F 0 "#PWR06" H 4700 5350 50  0001 C CNN
 F 1 "GND" H 4700 5450 50  0000 C CNN
 F 2 "" H 4700 5600 50  0001 C CNN
@@
 	4700 5500 4700 5600
 $Comp
-L +5V #PWR011
+L +5V #PWR07
 U 1 1 5B879F10
 P 4900 6000
-F 0 "#PWR011" H 4900 5850 50  0001 C CNN
+F 0 "#PWR07" H 4900 5850 50  0001 C CNN
 F 1 "+5V" H 4900 6140 50  0000 C CNN
 F 2 "" H 4900 6000 50  0001 C CNN
@@
 $EndComp
 $Comp
-L GND #PWR012
+L GND #PWR08
 U 1 1 5B879F3C
 P 4500 6700
-F 0 "#PWR012" H 4500 6450 50  0001 C CNN
+F 0 "#PWR08" H 4500 6450 50  0001 C CNN
 F 1 "GND" H 4500 6550 50  0000 C CNN
 F 2 "" H 4500 6700 50  0001 C CNN
@@
 Connection ~ 6200 6600
 $Comp
-L +3V3 #PWR013
+L +3V3 #PWR09
 U 1 1 5B87BEFA
 P 7600 6000
-F 0 "#PWR013" H 7600 5850 50  0001 C CNN
+F 0 "#PWR09" H 7600 5850 50  0001 C CNN
 F 1 "+3V3" H 7600 6140 50  0000 C CNN
 F 2 "" H 7600 6000 50  0001 C CNN
@@
 $EndComp
 $Comp
-L GND #PWR014
+L GND #PWR010
 U 1 1 5B87CC46
 P 5350 4100
-F 0 "#PWR014" H 5350 3850 50  0001 C CNN
+F 0 "#PWR010" H 5350 3850 50  0001 C CNN
 F 1 "GND" H 5350 3950 50  0000 C CNN
 F 2 "" H 5350 4100 50  0001 C CNN
@@
 $EndComp
 $Comp
-L GND #PWR015
+L GND #PWR011
 U 1 1 5B87D3B2
 P 3300 4900
-F 0 "#PWR015" H 3300 4650 50  0001 C CNN
+F 0 "#PWR011" H 3300 4650 50  0001 C CNN
 F 1 "GND" H 3300 4750 50  0000 C CNN
 F 2 "" H 3300 4900 50  0001 C CNN
@@
 $EndComp
 $Comp
-L +5V #PWR016
+L +5V #PWR012
 U 1 1 5B87D3F6
 P 3300 4400
-F 0 "#PWR016" H 3300 4250 50  0001 C CNN
+F 0 "#PWR012" H 3300 4250 50  0001 C CNN
 F 1 "+5V" H 3300 4540 50  0000 C CNN
 F 2 "" H 3300 4400 50  0001 C CNN
@@
 	3300 4800 3300 4900
 $Comp
-L PWR_FLAG #FLG017
+L PWR_FLAG #FLG013
 U 1 1 5B87DB70
 P 5200 6000
-F 0 "#FLG017" H 5200 6075 50  0001 C CNN
+F 0 "#FLG013" H 5200 6075 50  0001 C CNN
 F 1 "PWR_FLAG" H 5200 6150 50  0000 C CNN
 F 2 "" H 5200 6000 50  0001 C CNN
@@
 $EndComp
 $Comp
-L PWR_FLAG #FLG018
+L PWR_FLAG #FLG014
 U 1 1 5B87DBB4
 P 8000 6000
-F 0 "#FLG018" H 8000 6075 50  0001 C CNN
+F 0 "#FLG014" H 8000 6075 50  0001 C CNN
 F 1 "PWR_FLAG" H 8000 6150 50  0000 C CNN
 F 2 "" H 8000 6000 50  0001 C CNN
@@
 $EndComp
 $Comp
-L PWR_FLAG #FLG019
+L PWR_FLAG #FLG015
 U 1 1 5B87DBF8
 P 8000 6500
-F 0 "#FLG019" H 8000 6575 50  0001 C CNN
+F 0 "#FLG015" H 8000 6575 50  0001 C CNN
 F 1 "PWR_FLAG" H 8000 6650 50  0000 C CNN
 F 2 "" H 8000 6500 50  0001 C CNN
@@
 	6100 5000 6200 5000
 $Comp
-L R_POT_MountingPin RV?
+L R_POT_MountingPin RV1
 U 1 1 5B8B1245
 P 4650 3200
-F 0 "RV?" V 4475 3200 50  0000 C CNN
+F 0 "RV1" V 4475 3200 50  0000 C CNN
 F 1 "10K" V 4550 3200 50  0000 C CNN
 F 2 "" H 4650 3200 50  0001 C CNN
@@
 	4650 3050 4650 2900
 $Comp
-L GND #PWR?
+L GND #PWR016
 U 1 1 5B8B1B29
 P 4400 3300
-F 0 "#PWR?" H 4400 3050 50  0001 C CNN
+F 0 "#PWR016" H 4400 3050 50  0001 C CNN
 F 1 "GND" H 4400 3150 50  0000 C CNN
 F 2 "" H 4400 3300 50  0001 C CNN
@@
 Connection ~ 4400 3200
 $Comp
-L +3V3 #PWR?
+L +3V3 #PWR017
 U 1 1 5B8B1C95
 P 5000 3100
-F 0 "#PWR?" H 5000 2950 50  0001 C CNN
+F 0 "#PWR017" H 5000 2950 50  0001 C CNN
 F 1 "+3V3" H 5000 3240 50  0000 C CNN
 F 2 "" H 5000 3100 50  0001 C CNN
@@
 	5000 3200 5000 3100
 $Comp
-L R_POT_MountingPin RV?
+L R_POT_MountingPin RV2
 U 1 1 5B8B2593
 P 5850 3200
-F 0 "RV?" V 5675 3200 50  0000 C CNN
+F 0 "RV2" V 5675 3200 50  0000 C CNN
 F 1 "10K" V 5750 3200 50  0000 C CNN
 F 2 "" H 5850 3200 50  0001 C CNN
@@
 	5850 3050 5850 2900
 $Comp
-L GND #PWR?
+L GND #PWR018
 U 1 1 5B8B259B
 P 5600 3300
-F 0 "#PWR?" H 5600 3050 50  0001 C CNN
+F 0 "#PWR018" H 5600 3050 50  0001 C CNN
 F 1 "GND" H 5600 3150 50  0000 C CNN
 F 2 "" H 5600 3300 50  0001 C CNN
@@
 Connection ~ 5600 3200
 $Comp
-L +3V3 #PWR?
+L +3V3 #PWR019
 U 1 1 5B8B25A7
 P 6200 3100
-F 0 "#PWR?" H 6200 2950 50  0001 C CNN
+F 0 "#PWR019" H 6200 2950 50  0001 C CNN
 F 1 "+3V3" H 6200 3240 50  0000 C CNN
 F 2 "" H 6200 3100 50  0001 C CNN
@@
 Wire Wire Line
 	6200 3200 6200 3100
+NoConn ~ 7200 1200
+NoConn ~ 7200 1700
+NoConn ~ 7200 1800
+NoConn ~ 7200 1900
+NoConn ~ 7200 2000
+NoConn ~ 7200 2500
+NoConn ~ 7200 2600
+NoConn ~ 7200 2700
+NoConn ~ 7200 2800
+NoConn ~ 7200 2900
+NoConn ~ 7200 3400
+NoConn ~ 7200 3500
+NoConn ~ 7200 3600
+NoConn ~ 7200 3700
+NoConn ~ 7200 4400
+NoConn ~ 7200 4500
 $EndSCHEMATC

Commit message: Footprint for slide potentiometers.
Parts:
- RV1, RV2: footprint (none) -> footprints:Bourns_PTA4543
Changed lines of the file:
@@
 F 0 "RV1" V 4475 3200 50  0000 C CNN
 F 1 "10K" V 4550 3200 50  0000 C CNN
-F 2 "" H 4650 3200 50  0001 C CNN
+F 2 "footprints:Bourns_PTA4543" H 4650 3200 50  0001 C CNN
 F 3 "" H 4650 3200 50  0001 C CNN
 F 4 "PTA4553-2015CPB103" H 4650 3200 60  0001 C CNN "MPN"
@@
 F 0 "RV2" V 5675 3200 50  0000 C CNN
 F 1 "10K" V 5750 3200 50  0000 C CNN
-F 2 "" H 5850 3200 50  0001 C CNN
+F 2 "footprints:Bourns_PTA4543" H 5850 3200 50  0001 C CNN
 F 3 "" H 5850 3200 50  0001 C CNN
 F 4 "PTA4553-2015CPB103" H 5850 3200 60  0001 C CNN "MPN"

Commit message: I don't think we need that cap on 3V3.
Parts:
- removed C5: 47µF, Capacitors_THT:CP_Radial_D6.3mm_P2.50mm, symbol CP1
Changed lines of the file:
@@
 Wire Wire Line
 	7350 6100 8000 6100
-Wire Wire Line
-	7600 6000 7600 6200
-$Comp
-L CP1 C5
-U 1 1 5B87C55E
-P 7600 6350
-F 0 "C5" H 7625 6450 50  0000 L CNN
-F 1 "47µF" H 7625 6250 50  0000 L CNN
-F 2 "Capacitors_THT:CP_Radial_D6.3mm_P2.50mm" H 7638 6200 50  0001 C CNN
-F 3 "" H 7600 6350 50  0001 C CNN
-F 4 "ECE-A1CKS470" H 7600 6350 60  0001 C CNN "MPN"
-F 5 "CAP ALUM 47UF 20% 16V RADIAL" H 7600 6350 60  0001 C CNN "Description"
-F 6 "P969-ND" H 7600 6350 60  0001 C CNN "Digi-Key_PN"
-	1    7600 6350
-	1    0    0    -1
-$EndComp
 Connection ~ 7600 6100
-Wire Wire Line
-	7600 6600 7600 6500
 Connection ~ 6650 6600
 Wire Wire Line
@@
 Wire Wire Line
 	8000 6600 8000 6500
-Connection ~ 7600 6600
 $Comp
 L C C4
@@
 NoConn ~ 7200 4400
 NoConn ~ 7200 4500
+Wire Wire Line
+	7600 6000 7600 6100
 $EndSCHEMATC

Commit message: Add stuff on back silkscreen.
Other:
- note removed: "Check\nconnector\ndiameter!"
Changed lines of the file:
@@
 Sheet 1 1
 Title "Neopixel and potentiometer adapter for Micro:Bit"
-Date "2017-09-01"
-Rev ""
+Date "2017-09-03"
+Rev "1.0"
 Comp "Patrick Pelletier"
 Comment1 ""
@@
 	1    0    0    -1
 $EndComp
-Text Notes 3800 6350 0    60   ~ 0
-Check\nconnector\ndiameter!
 Wire Wire Line
 	6100 4650 6100 5000
