File: NeoBit.kicad_pcb (KiCad board)
At the start: 2 copper layers, 77.5 x 45.7 mm, 27 parts, among them J1 AudioJack3_Ground, J2 Barrel_Jack_MountingPin, J3 Qwiic, J4 DotStars, J5 microbit_edge_connector, J6 NeoPixels, U1 74AHCT125, U2 MCP1702-3302E_TO92, U3 MCP1702-5002E_TO92

Commit message: Finish wiring up PCB.
Parts:
- moved C8 2.16 mm to (182.6, 97.0), turned to 0 degrees
- moved C9 2.16 mm to (182.6, 102.9), turned to 0 degrees
Connections:
- C9 pad 1: Net-(C9-Pad1) -> Net-(C8-Pad1)
- C9 pad 2: Net-(C8-Pad2) -> Net-(C9-Pad2)
- J1 pad R: Net-(C9-Pad1) -> Net-(C9-Pad2)
- J1 pad T: Net-(C8-Pad1) -> Net-(C8-Pad2)
- R1 pad 1: Net-(C8-Pad2) -> Net-(C8-Pad1)
Routing:
- net /P0: track 9.93 -> 114.1 mm, vias 0 -> 2
- net Net-(C8-Pad2): track 0.00 -> 20.2 mm, vias 0 -> 1
- net Net-(C8-Pad1): track 0.00 -> 13.8 mm, vias 0 -> 1
- net Net-(C9-Pad2): track 0.00 -> 10.8 mm
- net Net-(C10-Pad1): track 0.00 -> 3.96 mm
Changed lines of the file:
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@@
   (general
     (links 87)
-    (no_connects 12)
+    (no_connects 1)
     (area 118.669999 83.744999 196.290001 129.615001)
     (thickness 1.6)
     (drawings 21)
-    (tracks 178)
+    (tracks 206)
     (zones 0)
     (modules 27)
@@
   (net 18 "Net-(C8-Pad1)")
   (net 19 "Net-(C8-Pad2)")
-  (net 20 "Net-(C9-Pad1)")
-  (net 21 "Net-(C10-Pad1)")
+  (net 20 "Net-(C10-Pad1)")
+  (net 21 "Net-(C9-Pad2)")
   (net_class Default "This is the default net class."
     (clearance 0.2)
@@
     (add_net "Net-(C8-Pad1)")
     (add_net "Net-(C8-Pad2)")
-    (add_net "Net-(C9-Pad1)")
+    (add_net "Net-(C9-Pad2)")
     (add_net "Net-(J6-Pad2)")
     (add_net "Net-(R2-Pad1)")
@@
     (descr "Terminal Block 4Ucon ItemNo. 10694, vertical (cable from top), 3 pins, pitch 3.5mm, size 11.5x8.3mm^2, drill diamater 1.3mm, pad diameter 2.6mm, see http://www.4uconnector.com/online/object/4udrawing/10694.pdf, script-generated with , script-generated using https://github.com/pointhi/kicad-footprint-generator/scripts/TerminalBlock_4Ucon")
     (tags "THT Terminal Block 4Ucon ItemNo. 10694 vertical pitch 3.5mm size 11.5x8.3mm^2 drill 1.3mm pad 2.6mm")
-    (fp_text reference J6 (at 9.144 -4.826 180) (layer F.SilkS)
+    (fp_text reference J6 (at 9.144 -4.572 180) (layer F.SilkS)
       (effects (font (size 1 1) (thickness 0.15)))
     )
@@
       (net 2 GND))
     (pad T thru_hole circle (at 2 2.4 270) (size 2.8 2.8) (drill 2) (layers *.Cu *.Mask)
-      (net 18 "Net-(C8-Pad1)"))
+      (net 19 "Net-(C8-Pad2)"))
     (pad R thru_hole circle (at 2 7.9 270) (size 2.8 2.8) (drill 2) (layers *.Cu *.Mask)
-      (net 20 "Net-(C9-Pad1)"))
+      (net 21 "Net-(C9-Pad2)"))
     (model ${KISYS3DMOD}/Connector_Audio.3dshapes/SJ1-3533NG.wrl
       (at (xyz 0 0 0))
@@
   )
   (module Capacitors_THT:CP_Radial_D5.0mm_P2.50mm (layer F.Cu)
-    (at 184.785 97.155 180)
+    (at 182.626 97.028)
     (descr "CP, Radial series, Radial, pin pitch=2.50mm, , diameter=5mm, Electrolytic Capacitor")
     (tags "CP Radial series Radial pin pitch 2.50mm  diameter 5mm Electrolytic Capacitor")
-    (fp_text reference C8 (at 3.683 -2.667 180) (layer F.SilkS)
-      (effects (font (size 1 1) (thickness 0.15)))
-    )
-    (fp_text value 220uF (at 1.25 3.81 180) (layer F.Fab)
+    (fp_text reference C8 (at -1.27 2.54) (layer F.SilkS)
+      (effects (font (size 1 1) (thickness 0.15)))
+    )
+    (fp_text value 220uF (at 1.25 3.81) (layer F.Fab)
       (effects (font (size 1 1) (thickness 0.15)))
     )
@@
     (fp_line (start 4.1 2.85) (end 4.1 -2.85) (layer F.CrtYd) (width 0.05))
     (fp_line (start 4.1 -2.85) (end -1.6 -2.85) (layer F.CrtYd) (width 0.05))
-    (fp_text user %R (at 1.25 0 180) (layer F.Fab)
-      (effects (font (size 1 1) (thickness 0.15)))
-    )
-    (pad 1 thru_hole rect (at 0 0 180) (size 1.6 1.6) (drill 0.8) (layers *.Cu *.Mask)
+    (fp_text user %R (at 1.25 0) (layer F.Fab)
+      (effects (font (size 1 1) (thickness 0.15)))
+    )
+    (pad 1 thru_hole rect (at 0 0) (size 1.6 1.6) (drill 0.8) (layers *.Cu *.Mask)
       (net 18 "Net-(C8-Pad1)"))
-    (pad 2 thru_hole circle (at 2.5 0 180) (size 1.6 1.6) (drill 0.8) (layers *.Cu *.Mask)
+    (pad 2 thru_hole circle (at 2.5 0) (size 1.6 1.6) (drill 0.8) (layers *.Cu *.Mask)
       (net 19 "Net-(C8-Pad2)"))
     (model ${KISYS3DMOD}/Capacitors_THT.3dshapes/CP_Radial_D5.0mm_P2.50mm.wrl
@@
   )
   (module Capacitors_THT:CP_Radial_D5.0mm_P2.50mm (layer F.Cu)
-    (at 184.785 102.87 180)
+    (at 182.626 102.87)
     (descr "CP, Radial series, Radial, pin pitch=2.50mm, , diameter=5mm, Electrolytic Capacitor")
     (tags "CP Radial series Radial pin pitch 2.50mm  diameter 5mm Electrolytic Capacitor")
-    (fp_text reference C9 (at 3.683 -2.794 180) (layer F.SilkS)
-      (effects (font (size 1 1) (thickness 0.15)))
-    )
-    (fp_text value 220uF (at 1.25 3.81 180) (layer F.Fab)
+    (fp_text reference C9 (at -1.27 2.54) (layer F.SilkS)
+      (effects (font (size 1 1) (thickness 0.15)))
+    )
+    (fp_text value 220uF (at 1.25 3.81) (layer F.Fab)
       (effects (font (size 1 1) (thickness 0.15)))
     )
@@
     (fp_line (start 4.1 2.85) (end 4.1 -2.85) (layer F.CrtYd) (width 0.05))
     (fp_line (start 4.1 -2.85) (end -1.6 -2.85) (layer F.CrtYd) (width 0.05))
-    (fp_text user %R (at 1.25 0 180) (layer F.Fab)
-      (effects (font (size 1 1) (thickness 0.15)))
-    )
-    (pad 1 thru_hole rect (at 0 0 180) (size 1.6 1.6) (drill 0.8) (layers *.Cu *.Mask)
-      (net 20 "Net-(C9-Pad1)"))
-    (pad 2 thru_hole circle (at 2.5 0 180) (size 1.6 1.6) (drill 0.8) (layers *.Cu *.Mask)
-      (net 19 "Net-(C8-Pad2)"))
+    (fp_text user %R (at 1.25 0) (layer F.Fab)
+      (effects (font (size 1 1) (thickness 0.15)))
+    )
+    (pad 1 thru_hole rect (at 0 0) (size 1.6 1.6) (drill 0.8) (layers *.Cu *.Mask)
+      (net 18 "Net-(C8-Pad1)"))
+    (pad 2 thru_hole circle (at 2.5 0) (size 1.6 1.6) (drill 0.8) (layers *.Cu *.Mask)
+      (net 21 "Net-(C9-Pad2)"))
     (model ${KISYS3DMOD}/Capacitors_THT.3dshapes/CP_Radial_D5.0mm_P2.50mm.wrl
       (at (xyz 0 0 0))
@@
     )
     (pad 1 thru_hole circle (at 0 0 90) (size 1.6 1.6) (drill 0.8) (layers *.Cu *.Mask)
-      (net 21 "Net-(C10-Pad1)"))
+      (net 20 "Net-(C10-Pad1)"))
     (pad 2 thru_hole circle (at 2.5 0 90) (size 1.6 1.6) (drill 0.8) (layers *.Cu *.Mask)
       (net 2 GND))
@@
     (fp_line (start 3.65 -1.6) (end -1.6 -1.6) (layer F.CrtYd) (width 0.05))
     (pad 1 thru_hole circle (at 0 0) (size 1.6 1.6) (drill 0.8) (layers *.Cu *.Mask)
-      (net 19 "Net-(C8-Pad2)"))
+      (net 18 "Net-(C8-Pad1)"))
     (pad 2 thru_hole oval (at 2.54 0) (size 1.6 1.6) (drill 0.8) (layers *.Cu *.Mask)
       (net 5 /P0))
@@
     (fp_line (start 3.65 -1.6) (end -1.6 -1.6) (layer F.CrtYd) (width 0.05))
     (pad 1 thru_hole circle (at 0 0) (size 1.6 1.6) (drill 0.8) (layers *.Cu *.Mask)
-      (net 21 "Net-(C10-Pad1)"))
+      (net 20 "Net-(C10-Pad1)"))
     (pad 2 thru_hole oval (at 2.54 0) (size 1.6 1.6) (drill 0.8) (layers *.Cu *.Mask)
       (net 5 /P0))
@@
   (segment (start 164.465 107.315) (end 164.465 97.79) (width 0.508) (layer B.Cu) (net 4) (status 10))
   (via (at 164.465 97.79) (size 0.6) (drill 0.4) (layers F.Cu B.Cu) (net 4))
+  (segment (start 179.705 107.315) (end 179.705 108.44637) (width 0.25) (layer B.Cu) (net 5))
+  (segment (start 179.705 108.44637) (end 180.504999 109.246369) (width 0.25) (layer B.Cu) (net 5))
+  (segment (start 180.504999 109.246369) (end 180.504999 115.405001) (width 0.25) (layer B.Cu) (net 5))
+  (segment (start 180.504999 115.405001) (end 179.705 116.205) (width 0.25) (layer B.Cu) (net 5))
+  (segment (start 176.784 123.444) (end 176.784 119.126) (width 0.25) (layer B.Cu) (net 5))
+  (segment (start 176.784 119.126) (end 179.705 116.205) (width 0.25) (layer B.Cu) (net 5))
+  (segment (start 123.19 123.444) (end 176.784 123.444) (width 0.25) (layer F.Cu) (net 5))
+  (via (at 176.784 123.444) (size 0.6) (drill 0.4) (layers F.Cu B.Cu) (net 5))
+  (segment (start 124.46 91.44) (end 123.124999 92.775001) (width 0.25) (layer B.Cu) (net 5))
+  (segment (start 123.124999 92.775001) (end 123.124999 123.378999) (width 0.25) (layer B.Cu) (net 5))
+  (segment (start 123.124999 123.378999) (end 123.19 123.444) (width 0.25) (layer B.Cu) (net 5))
+  (via (at 123.19 123.444) (size 0.6) (drill 0.4) (layers F.Cu B.Cu) (net 5))
   (segment (start 124.46 91.44) (end 127 91.44) (width 0.25) (layer F.Cu) (net 5) (status 30))
   (segment (start 125.73 89.54) (end 128.27 89.54) (width 0.25) (layer F.Cu) (net 5) (status 30))
@@
   (segment (start 184.77 92.695) (end 184.785 92.71) (width 0.25) (layer B.Cu) (net 17))
   (via (at 184.785 92.71) (size 0.6) (drill 0.4) (layers F.Cu B.Cu) (net 17))
+  (segment (start 180.34 104.775) (end 179.705 104.775) (width 0.25) (layer F.Cu) (net 18))
+  (segment (start 179.705 104.775) (end 177.165 107.315) (width 0.25) (layer F.Cu) (net 18))
+  (segment (start 182.626 102.87) (end 182.626 103.92) (width 0.25) (layer B.Cu) (net 18))
+  (segment (start 182.626 103.92) (end 181.771 104.775) (width 0.25) (layer B.Cu) (net 18))
+  (segment (start 181.771 104.775) (end 180.34 104.775) (width 0.25) (layer B.Cu) (net 18))
+  (via (at 180.34 104.775) (size 0.6) (drill 0.4) (layers F.Cu B.Cu) (net 18))
+  (segment (start 182.626 97.028) (end 182.626 102.87) (width 0.25) (layer B.Cu) (net 18))
+  (segment (start 187.035 110.49) (end 189.275 110.49) (width 0.25) (layer F.Cu) (net 19))
+  (segment (start 189.275 110.49) (end 191.91 113.125) (width 0.25) (layer F.Cu) (net 19))
+  (segment (start 185.126 97.028) (end 187.035 98.937) (width 0.25) (layer B.Cu) (net 19))
+  (segment (start 187.035 98.937) (end 187.035 110.49) (width 0.25) (layer B.Cu) (net 19))
+  (via (at 187.035 110.49) (size 0.6) (drill 0.4) (layers F.Cu B.Cu) (net 19))
+  (segment (start 177.165 116.205) (end 179.07 114.3) (width 0.25) (layer B.Cu) (net 20))
+  (segment (start 179.07 114.3) (end 179.07 113.03) (width 0.25) (layer B.Cu) (net 20))
+  (segment (start 186.41 113.125) (end 186.41 104.154) (width 0.25) (layer B.Cu) (net 21))
+  (segment (start 186.41 104.154) (end 185.126 102.87) (width 0.25) (layer B.Cu) (net 21))
   (zone (net 9) (net_name +VDC) (layer F.Cu) (hatch edge 0.508)
     (priority 1)

Commit message: Passing DRC now.
Routing:
- net Net-(R2-Pad1): track 18.9 -> 21.1 mm
Changed lines of the file:
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@@
   (general
     (links 87)
-    (no_connects 1)
-    (area 118.669999 83.744999 196.290001 129.615001)
+    (no_connects 0)
+    (area 117.08 69.365 200.235001 131.993096)
     (thickness 1.6)
     (drawings 21)
-    (tracks 206)
+    (tracks 210)
     (zones 0)
     (modules 27)
@@
   (segment (start 146.375 125.42) (end 146.685 125.73) (width 0.25) (layer F.Cu) (net 7))
   (via (at 146.685 125.73) (size 0.6) (drill 0.4) (layers F.Cu B.Cu) (net 7))
-  (segment (start 145.415 111.98) (end 145.415 106.045) (width 0.25) (layer B.Cu) (net 8))
+  (segment (start 144.403073 112.436184) (end 144.103074 112.136185) (width 0.25) (layer F.Cu) (net 8))
+  (segment (start 156.98363 111.76) (end 156.307446 112.436184) (width 0.25) (layer F.Cu) (net 8))
   (segment (start 158.115 111.76) (end 156.98363 111.76) (width 0.25) (layer F.Cu) (net 8))
-  (segment (start 156.98363 111.76) (end 156.493629 112.250001) (width 0.25) (layer F.Cu) (net 8))
-  (via (at 145.415 111.98) (size 0.6) (drill 0.4) (layers F.Cu B.Cu) (net 8))
-  (segment (start 156.493629 112.250001) (end 145.685001 112.250001) (width 0.25) (layer F.Cu) (net 8))
-  (segment (start 145.685001 112.250001) (end 145.415 111.98) (width 0.25) (layer F.Cu) (net 8))
+  (segment (start 144.403073 111.836186) (end 144.103074 112.136185) (width 0.25) (layer B.Cu) (net 8))
+  (segment (start 156.307446 112.436184) (end 144.403073 112.436184) (width 0.25) (layer F.Cu) (net 8))
+  (segment (start 145.415 110.824259) (end 144.403073 111.836186) (width 0.25) (layer B.Cu) (net 8))
+  (segment (start 145.415 106.045) (end 145.415 110.824259) (width 0.25) (layer B.Cu) (net 8))
+  (via (at 144.103074 112.136185) (size 0.6) (drill 0.4) (layers F.Cu B.Cu) (net 8))
   (segment (start 163.83 114.3) (end 159.016 114.3) (width 0.508) (layer F.Cu) (net 9))
   (segment (start 159.016 114.3) (end 159.004 114.312) (width 0.508) (layer F.Cu) (net 9))
@@
   (via (at 180.34 104.775) (size 0.6) (drill 0.4) (layers F.Cu B.Cu) (net 18))
   (segment (start 182.626 97.028) (end 182.626 102.87) (width 0.25) (layer B.Cu) (net 18))
-  (segment (start 187.035 110.49) (end 189.275 110.49) (width 0.25) (layer F.Cu) (net 19))
-  (segment (start 189.275 110.49) (end 191.91 113.125) (width 0.25) (layer F.Cu) (net 19))
-  (segment (start 185.126 97.028) (end 187.035 98.937) (width 0.25) (layer B.Cu) (net 19))
-  (segment (start 187.035 98.937) (end 187.035 110.49) (width 0.25) (layer B.Cu) (net 19))
-  (via (at 187.035 110.49) (size 0.6) (drill 0.4) (layers F.Cu B.Cu) (net 19))
+  (segment (start 187.435969 110.084932) (end 187.435969 110.509196) (width 0.25) (layer B.Cu) (net 19))
+  (segment (start 187.435969 99.337969) (end 187.435969 110.084932) (width 0.25) (layer B.Cu) (net 19))
+  (segment (start 185.126 97.028) (end 187.435969 99.337969) (width 0.25) (layer B.Cu) (net 19))
+  (segment (start 189.294196 110.509196) (end 187.860233 110.509196) (width 0.25) (layer F.Cu) (net 19))
+  (segment (start 191.91 113.125) (end 189.294196 110.509196) (width 0.25) (layer F.Cu) (net 19))
+  (segment (start 187.860233 110.509196) (end 187.435969 110.509196) (width 0.25) (layer F.Cu) (net 19))
+  (via (at 187.435969 110.509196) (size 0.6) (drill 0.4) (layers F.Cu B.Cu) (net 19))
   (segment (start 177.165 116.205) (end 179.07 114.3) (width 0.25) (layer B.Cu) (net 20))
   (segment (start 179.07 114.3) (end 179.07 113.03) (width 0.25) (layer B.Cu) (net 20))
